Commit message: :bento: Unify on using livox_joint & livox_link; remove redundent collision stuff

File: ros_assets/h1_2_handless_ros.urdf (robot description, URDF)
Before this commit: robot h1_2, 35 links, 34 joints
Links:
- removed link head_camera_link
- removed link left_hand_camera_link
- removed link lidar_link
- removed link right_hand_camera_link
- added link livox_link
Joints:
- removed joint head_camera_joint
- removed joint left_hand_camera_joint
- removed joint lidar_joint
- removed joint right_hand_camera_joint
- added joint livox_joint: type fixed, parent torso_link, child livox_link, origin xyz=0.04874 0 0.67980 rpy=0 0.24015730507441985 0

File: ros_assets/h1_2_magpie_homie.urdf (robot description, URDF)
Before this commit: robot h1_2, 34 links, 33 joints
Links:
- removed link lidar_link
- added link livox_link
Joints:
- removed joint lidar_joint
- added joint livox_joint: type fixed, parent torso_link, child livox_link, origin xyz=0.04874 0 0.67980 rpy=0 0.24015730507441985 0

File: ros_assets/h1_2_magpie_ros.urdf (robot description, URDF)
Before this commit: robot h1_2_magpie, 53 links, 52 joints
Links:
- removed link head_camera_link
- removed link left_hand_camera_link
- removed link lidar_link
- removed link right_hand_camera_link
- added link livox_link
Joints:
- removed joint head_camera_joint
- removed joint left_hand_camera_joint
- removed joint lidar_joint
- removed joint right_hand_camera_joint
- added joint livox_joint: type fixed, parent torso_link, child livox_link, origin xyz=0.04874 0 0.67980 rpy=0 0.24015730507441985 0
