Commit message: add hand in eye cameras

File: ros_assets/h1_2_handless.urdf (robot description, URDF)
Before this commit: robot h1_2, 32 links, 31 joints
Links:
- added link left_grip_site, mass 1e-6
- added link right_grip_site, mass 1e-6
Joints:
- added joint left_grip_site_joint: type fixed, parent left_wrist_yaw_link, child left_grip_site, origin xyz=0.272 0 0.000875 rpy=0 0 0
- added joint right_grip_site_joint: type fixed, parent right_wrist_yaw_link, child right_grip_site, origin xyz=0.272 0 0.000875 rpy=0 0 0

Commit message: :bento: Update shoulder_roll_joint limits in all descriptions to match the new hardware

File: ros_assets/h1_2_handless.urdf (robot description, URDF)
Before this commit: robot h1_2, 34 links, 33 joints
Joints:
- joint left_shoulder_roll_joint: limit lower=-0.38 upper=3.4 effort=40 velocity=9 -> lower=-0.19 upper=3.4 effort=40 velocity=9
- joint right_shoulder_roll_joint: limit lower=-3.4 upper=0.38 effort=40 velocity=9 -> lower=-3.4 upper=0.19 effort=40 velocity=9

File: ros_assets/h1_2_handless_ros.urdf (robot description, URDF)
Before this commit: robot h1_2, 35 links, 34 joints
Joints:
- joint left_shoulder_roll_joint: limit lower=-0.38 upper=3.4 effort=40 velocity=9 -> lower=-0.19 upper=3.4 effort=40 velocity=9
- joint right_shoulder_roll_joint: limit lower=-3.4 upper=0.38 effort=40 velocity=9 -> lower=-3.4 upper=0.19 effort=40 velocity=9

File: ros_assets/h1_2_magpie.urdf (robot description, URDF)
Before this commit: robot h1_2_magpie, 50 links, 49 joints
Joints:
- joint left_shoulder_roll_joint: limit lower=-0.38 upper=3.4 effort=40 velocity=9 -> lower=-0.19 upper=3.4 effort=40 velocity=9
- joint right_shoulder_roll_joint: limit lower=-3.4 upper=0.38 effort=40 velocity=9 -> lower=-3.4 upper=0.19 effort=40 velocity=9

File: ros_assets/h1_2_magpie_homie.urdf (robot description, URDF)
Before this commit: robot h1_2, 34 links, 33 joints
Joints:
- joint left_shoulder_roll_joint: limit lower=-0.38 upper=3.4 effort=40 velocity=9 -> lower=-0.19 upper=3.4 effort=40 velocity=9
- joint right_shoulder_roll_joint: limit lower=-3.4 upper=0.38 effort=40 velocity=9 -> lower=-3.4 upper=0.19 effort=40 velocity=9

File: ros_assets/h1_2_magpie_ros.urdf (robot description, URDF)
Before this commit: robot h1_2_magpie, 53 links, 52 joints
Joints:
- joint left_shoulder_roll_joint: limit lower=-0.38 upper=3.4 effort=40 velocity=9 -> lower=-0.19 upper=3.4 effort=40 velocity=9
- joint right_shoulder_roll_joint: limit lower=-3.4 upper=0.38 effort=40 velocity=9 -> lower=-3.4 upper=0.19 effort=40 velocity=9

Commit message: :sparkles: Add left_grasp_frame & right_grasp_frame for MAGPIE gripper closing point

File: ros_assets/h1_2_handless.urdf (robot description, URDF)
Before this commit: robot h1_2, 34 links, 33 joints
Links:
- removed link left_grip_site
- removed link right_grip_site
- added link left_grasp_frame, mass 1e-6
- added link right_grasp_frame, mass 1e-6
Joints:
- removed joint left_grip_site_joint
- removed joint right_grip_site_joint
- added joint left_grasp_frame_joint: type fixed, parent left_wrist_yaw_link, child left_grasp_frame, origin xyz=0.231991 0 0.000625 rpy=0 0 0
- added joint right_grasp_frame_joint: type fixed, parent right_wrist_yaw_link, child right_grasp_frame, origin xyz=0.231991 0 0.000625 rpy=0 0 0

File: ros_assets/h1_2_handless_ros.urdf (robot description, URDF)
Before this commit: robot h1_2, 32 links, 31 joints
Links:
- added link left_grasp_frame, mass 1e-6
- added link right_grasp_frame, mass 1e-6
Joints:
- added joint left_grasp_frame_joint: type fixed, parent left_wrist_yaw_link, child left_grasp_frame, origin xyz=0.231991 0 0.000625 rpy=0 0 0
- added joint right_grasp_frame_joint: type fixed, parent right_wrist_yaw_link, child right_grasp_frame, origin xyz=0.231991 0 0.000625 rpy=0 0 0

File: ros_assets/h1_2_magpie.urdf (robot description, URDF)
Before this commit: robot h1_2_magpie, 50 links, 49 joints
Links:
- added link left_grasp_frame, mass 1e-6
- added link right_grasp_frame, mass 1e-6
Joints:
- added joint left_grasp_frame_joint: type fixed, parent left_wrist_yaw_link, child left_grasp_frame, origin xyz=0.231991 0 0.000625 rpy=0 0 0
- added joint right_grasp_frame_joint: type fixed, parent right_wrist_yaw_link, child right_grasp_frame, origin xyz=0.231991 0 0.000625 rpy=0 0 0

File: ros_assets/h1_2_magpie_homie.urdf (robot description, URDF)
Before this commit: robot h1_2, 34 links, 33 joints
Links:
- added link left_grasp_frame, mass 1e-6
- added link right_grasp_frame, mass 1e-6
Joints:
- added joint left_grasp_frame_joint: type fixed, parent left_wrist_yaw_link, child left_grasp_frame, origin xyz=0.231991 0 0.000625 rpy=0 0 0
- added joint right_grasp_frame_joint: type fixed, parent right_wrist_yaw_link, child right_grasp_frame, origin xyz=0.231991 0 0.000625 rpy=0 0 0

File: ros_assets/h1_2_magpie_ros.urdf (robot description, URDF)
Before this commit: robot h1_2_magpie, 50 links, 49 joints
Links:
- added link left_grasp_frame, mass 1e-6
- added link right_grasp_frame, mass 1e-6
Joints:
- added joint left_grasp_frame_joint: type fixed, parent left_wrist_yaw_link, child left_grasp_frame, origin xyz=0.231991 0 0.000625 rpy=0 0 0
- added joint right_grasp_frame_joint: type fixed, parent right_wrist_yaw_link, child right_grasp_frame, origin xyz=0.231991 0 0.000625 rpy=0 0 0

Commit message: fix graspgenx frames woohoo

File: ros_assets/h1_2_handless.urdf (robot description, URDF)
Before this commit: robot h1_2, 34 links, 33 joints
Links:
- added link left_graspgenx_frame, mass 1e-6
- added link right_graspgenx_frame, mass 1e-6
Joints:
- added joint left_graspgen_frame_joint: type fixed, parent left_wrist_yaw_link, child left_graspgenx_frame, origin xyz=0.0 0 0.0 rpy=1.5708 0 1.5708
- added joint right_graspgen_frame_joint: type fixed, parent right_wrist_yaw_link, child right_graspgenx_frame, origin xyz=0.0 0 0.0 rpy=1.5708 0 1.5708

File: ros_assets/h1_2_handless_ros.urdf (robot description, URDF)
Before this commit: robot h1_2, 34 links, 33 joints
Links:
- added link left_graspgenx_frame, mass 1e-6
- added link right_graspgenx_frame, mass 1e-6
Joints:
- added joint left_graspgen_frame_joint: type fixed, parent left_wrist_yaw_link, child left_graspgenx_frame, origin xyz=0.0 0 0.0 rpy=1.5708 0 1.5708
- added joint right_graspgen_frame_joint: type fixed, parent right_wrist_yaw_link, child right_graspgenx_frame, origin xyz=0.0 0 0.0 rpy=1.5708 0 1.5708

File: ros_assets/h1_2_magpie.urdf (robot description, URDF)
Before this commit: robot h1_2_magpie, 52 links, 51 joints
Links:
- added link left_graspgenx_frame, mass 1e-6
- added link right_graspgenx_frame, mass 1e-6
Joints:
- added joint left_graspgenx_frame_joint: type fixed, parent left_wrist_yaw_link, child left_graspgenx_frame, origin xyz=0.0 0 0.0000 rpy=1.5708 0 1.5708
- added joint right_graspgenx_frame_joint: type fixed, parent right_wrist_yaw_link, child right_graspgenx_frame, origin xyz=0.0 0 0.000 rpy=1.5708 0 1.5708 

File: ros_assets/h1_2_magpie_ros.urdf (robot description, URDF)
Before this commit: robot h1_2_magpie, 52 links, 51 joints
Links:
- added link left_graspgenx_frame, mass 1e-6
- added link right_graspgenx_frame, mass 1e-6
Joints:
- added joint left_graspgenx_frame_joint: type fixed, parent left_wrist_yaw_link, child left_graspgenx_frame, origin xyz=0.0 0 0.0000 rpy=1.5708 0 1.5708
- added joint right_graspgenx_frame_joint: type fixed, parent right_wrist_yaw_link, child right_graspgenx_frame, origin xyz=0.0 0 0.000 rpy=1.5708 0 1.5708 
- joint lg_left_hinge_1: axis 1 0 0 -> (none); limit lower=-0.035 upper=2.05 effort=10 velocity=3.14 -> (none); type revolute -> fixed
- joint lg_left_hinge_2: axis 1 0 0 -> (none); type continuous -> fixed
- joint lg_left_hinge_3: axis 1 0 0 -> (none); type continuous -> fixed
- joint lg_right_hinge_1: axis 1 0 0 -> (none); limit lower=-2.05 upper=0.035 effort=10 velocity=3.14 -> (none); type revolute -> fixed
- joint lg_right_hinge_2: axis 1 0 0 -> (none); type continuous -> fixed
- joint lg_right_hinge_3: axis 1 0 0 -> (none); type continuous -> fixed
- joint rg_left_hinge_1: axis 1 0 0 -> (none); limit lower=-0.035 upper=2.05 effort=10 velocity=3.14 -> (none); type revolute -> fixed
- joint rg_left_hinge_2: axis 1 0 0 -> (none); type continuous -> fixed
- joint rg_left_hinge_3: axis 1 0 0 -> (none); type continuous -> fixed
- joint rg_right_hinge_1: axis 1 0 0 -> (none); limit lower=-2.05 upper=0.035 effort=10 velocity=3.14 -> (none); type revolute -> fixed
- joint rg_right_hinge_2: axis 1 0 0 -> (none); type continuous -> fixed
- joint rg_right_hinge_3: axis 1 0 0 -> (none); type continuous -> fixed

Commit message: update graspgenx frame offset

File: ros_assets/h1_2_handless.urdf (robot description, URDF)
Before this commit: robot h1_2, 36 links, 35 joints
Joints:
- joint left_graspgen_frame_joint: origin xyz=0.0 0 0.0 rpy=1.5708 0 1.5708 -> xyz=0.117415 0 -0.001613 rpy=1.5708 0 1.5708
- joint right_graspgen_frame_joint: origin xyz=0.0 0 0.0 rpy=1.5708 0 1.5708 -> xyz=0.117415 0 -0.001613 rpy=1.5708 0 1.5708

File: ros_assets/h1_2_handless_ros.urdf (robot description, URDF)
Before this commit: robot h1_2, 36 links, 35 joints
Joints:
- joint left_graspgen_frame_joint: origin xyz=0.0 0 0.0 rpy=1.5708 0 1.5708 -> xyz=0.117415 0 -0.001613 rpy=1.5708 0 1.5708
- joint right_graspgen_frame_joint: origin xyz=0.0 0 0.0 rpy=1.5708 0 1.5708 -> xyz=0.117415 0 -0.001613 rpy=1.5708 0 1.5708

File: ros_assets/h1_2_magpie.urdf (robot description, URDF)
Before this commit: robot h1_2_magpie, 54 links, 53 joints
Joints:
- joint left_graspgenx_frame_joint: origin xyz=0.0 0 0.0000 rpy=1.5708 0 1.5708 -> xyz=0.117415 0 -0.001613 rpy=1.5708 0 1.5708
- joint right_graspgenx_frame_joint: origin xyz=0.0 0 0.000 rpy=1.5708 0 1.5708  -> xyz=0.117415 0 -0.001613 rpy=1.5708 0 1.5708

File: ros_assets/h1_2_magpie_ros.urdf (robot description, URDF)
Before this commit: robot h1_2_magpie, 54 links, 53 joints
Joints:
- joint left_graspgenx_frame_joint: origin xyz=0.0 0 0.0000 rpy=1.5708 0 1.5708 -> xyz=0.117415 0 -0.001613 rpy=1.5708 0 1.5708
- joint right_graspgenx_frame_joint: origin xyz=0.0 0 0.000 rpy=1.5708 0 1.5708  -> xyz=0.117415 0 -0.001613 rpy=1.5708 0 1.5708

Commit message: flip grasp frame orientation seems to have worked

File: ros_assets/h1_2_handless.urdf (robot description, URDF)
Before this commit: robot h1_2, 36 links, 35 joints
Joints:
- joint left_graspgen_frame_joint: origin xyz=0.117415 0 -0.001613 rpy=1.5708 0 1.5708 -> xyz=0.117415 0 -0.001613 rpy=-1.5708 0 -1.5708
- joint right_graspgen_frame_joint: origin xyz=0.117415 0 -0.001613 rpy=1.5708 0 1.5708 -> xyz=0.117415 0 -0.001613 rpy=-1.5708 0 -1.5708

File: ros_assets/h1_2_handless_ros.urdf (robot description, URDF)
Before this commit: robot h1_2, 36 links, 35 joints
Joints:
- joint left_graspgen_frame_joint: origin xyz=0.117415 0 -0.001613 rpy=1.5708 0 1.5708 -> xyz=0.117415 0 -0.001613 rpy=-1.5708 0 -1.5708
- joint right_graspgen_frame_joint: origin xyz=0.117415 0 -0.001613 rpy=1.5708 0 1.5708 -> xyz=0.117415 0 -0.001613 rpy=-1.5708 0 -1.5708

File: ros_assets/h1_2_magpie.urdf (robot description, URDF)
Before this commit: robot h1_2_magpie, 54 links, 53 joints
Joints:
- joint left_graspgenx_frame_joint: origin xyz=0.117415 0 -0.001613 rpy=1.5708 0 1.5708 -> xyz=0.117415 0 -0.001613 rpy=-1.5708 0 -1.5708
- joint right_graspgenx_frame_joint: origin xyz=0.117415 0 -0.001613 rpy=1.5708 0 1.5708 -> xyz=0.117415 0 -0.001613 rpy=-1.5708 0 -1.5708

File: ros_assets/h1_2_magpie_ros.urdf (robot description, URDF)
Before this commit: robot h1_2_magpie, 54 links, 53 joints
Joints:
- joint left_graspgenx_frame_joint: origin xyz=0.117415 0 -0.001613 rpy=1.5708 0 1.5708 -> xyz=0.117415 0 -0.001613 rpy=-1.5708 0 -1.5708
- joint right_graspgenx_frame_joint: origin xyz=0.117415 0 -0.001613 rpy=1.5708 0 1.5708 -> xyz=0.117415 0 -0.001613 rpy=-1.5708 0 -1.5708

Commit message: Flip graspgenx frames again

File: ros_assets/h1_2_handless.urdf (robot description, URDF)
Before this commit: robot h1_2, 36 links, 35 joints
Joints:
- removed joint left_graspgen_frame_joint
- removed joint right_graspgen_frame_joint
- added joint left_graspgenx_frame_joint: type fixed, parent left_wrist_yaw_link, child left_graspgenx_frame, origin xyz=0.117415 0 -0.001613 rpy=1.5708 0 1.5708
- added joint right_graspgenx_frame_joint: type fixed, parent right_wrist_yaw_link, child right_graspgenx_frame, origin xyz=0.117415 0 -0.001613 rpy=1.5708 0 1.5708

File: ros_assets/h1_2_handless_ros.urdf (robot description, URDF)
Before this commit: robot h1_2, 36 links, 35 joints
Joints:
- removed joint left_graspgen_frame_joint
- removed joint right_graspgen_frame_joint
- added joint left_graspgenx_frame_joint: type fixed, parent left_wrist_yaw_link, child left_graspgenx_frame, origin xyz=0.117415 0 -0.001613 rpy=1.5708 0 1.5708
- added joint right_graspgenx_frame_joint: type fixed, parent right_wrist_yaw_link, child right_graspgenx_frame, origin xyz=0.117415 0 -0.001613 rpy=1.5708 0 1.5708

File: ros_assets/h1_2_magpie.urdf (robot description, URDF)
Before this commit: robot h1_2_magpie, 54 links, 53 joints
Joints:
- joint left_graspgenx_frame_joint: origin xyz=0.117415 0 -0.001613 rpy=-1.5708 0 -1.5708 -> xyz=0.117415 0 -0.001613 rpy=1.5708 0 1.5708
- joint right_graspgenx_frame_joint: origin xyz=0.117415 0 -0.001613 rpy=-1.5708 0 -1.5708 -> xyz=0.117415 0 -0.001613 rpy=1.5708 0 1.5708

File: ros_assets/h1_2_magpie_ros.urdf (robot description, URDF)
Before this commit: robot h1_2_magpie, 54 links, 53 joints
Joints:
- joint left_graspgenx_frame_joint: origin xyz=0.117415 0 -0.001613 rpy=-1.5708 0 -1.5708 -> xyz=0.117415 0 -0.001613 rpy=1.5708 0 1.5708
- joint right_graspgenx_frame_joint: origin xyz=0.117415 0 -0.001613 rpy=-1.5708 0 -1.5708 -> xyz=0.117415 0 -0.001613 rpy=1.5708 0 1.5708

Commit message: tune graspgen frames

File: ros_assets/h1_2_handless.urdf (robot description, URDF)
Before this commit: robot h1_2, 36 links, 35 joints
Joints:
- joint left_graspgenx_frame_joint: origin xyz=0.117415 0 -0.001613 rpy=1.5708 0 1.5708 -> xyz=0.085  0 -0.001613 rpy=1.5708 0 1.5708
- joint right_graspgenx_frame_joint: origin xyz=0.117415 0 -0.001613 rpy=1.5708 0 1.5708 -> xyz=0.085  0 -0.001613 rpy=1.5708 0 1.5708

File: ros_assets/h1_2_handless_ros.urdf (robot description, URDF)
Before this commit: robot h1_2, 36 links, 35 joints
Joints:
- joint left_graspgenx_frame_joint: origin xyz=0.117415 0 -0.001613 rpy=1.5708 0 1.5708 -> xyz=0.085  0 -0.001613 rpy=1.5708 0 1.5708
- joint right_graspgenx_frame_joint: origin xyz=0.117415 0 -0.001613 rpy=1.5708 0 1.5708 -> xyz=0.085  0 -0.001613 rpy=1.5708 0 1.5708

File: ros_assets/h1_2_magpie.urdf (robot description, URDF)
Before this commit: robot h1_2_magpie, 54 links, 53 joints
Joints:
- joint left_graspgenx_frame_joint: origin xyz=0.117415 0 -0.001613 rpy=1.5708 0 1.5708 -> xyz=0.085 0 -0.001613 rpy=1.5708 0 1.5708
- joint right_graspgenx_frame_joint: origin xyz=0.117415 0 -0.001613 rpy=1.5708 0 1.5708 -> xyz=0.085 0 -0.001613 rpy=1.5708 0 1.5708

File: ros_assets/h1_2_magpie_ros.urdf (robot description, URDF)
Before this commit: robot h1_2_magpie, 54 links, 53 joints
Joints:
- joint left_graspgenx_frame_joint: origin xyz=0.117415 0 -0.001613 rpy=1.5708 0 1.5708 -> xyz=0.085 0 -0.001613 rpy=1.5708 0 1.5708
- joint right_graspgenx_frame_joint: origin xyz=0.117415 0 -0.001613 rpy=1.5708 0 1.5708 -> xyz=0.085 0 -0.001613 rpy=1.5708 0 1.5708

Commit message: add head camera link back in

File: ros_assets/h1_2_handless.urdf (robot description, URDF)
Before this commit: robot h1_2, 36 links, 35 joints
Links:
- removed link camera_link
- added link head_camera_link
Joints:
- removed joint camera_joint
- added joint head_camera_joint: type fixed, parent torso_link, child head_camera_link, origin xyz=0.11109 0.01750 0.68789 rpy=-2.45672546 0 -1.5708

File: ros_assets/h1_2_handless_ros.urdf (robot description, URDF)
Before this commit: robot h1_2, 36 links, 35 joints
Links:
- removed link camera_link
- added link head_camera_link
Joints:
- removed joint camera_joint
- added joint head_camera_joint: type fixed, parent torso_link, child head_camera_link, origin xyz=0.11109 0.01750 0.68789 rpy=-2.45672546 0 -1.5708

File: ros_assets/h1_2_magpie.urdf (robot description, URDF)
Before this commit: robot h1_2_magpie, 54 links, 53 joints
Links:
- removed link camera_link
- added link head_camera_link
Joints:
- removed joint camera_joint
- added joint head_camera_joint: type fixed, parent torso_link, child head_camera_link, origin xyz=0.11109 0.01750 0.68789 rpy=-2.45672546 0 -1.5708

File: ros_assets/h1_2_magpie_homie.urdf (robot description, URDF)
Before this commit: robot h1_2, 36 links, 35 joints
Links:
- removed link camera_link
- added link head_camera_link
Joints:
- removed joint camera_joint
- added joint head_camera_joint: type fixed, parent torso_link, child head_camera_link, origin xyz=0.11109 0.01750 0.68789 rpy=-2.45672546 0 -1.5708

File: ros_assets/h1_2_magpie_ros.urdf (robot description, URDF)
Before this commit: robot h1_2_magpie, 54 links, 53 joints
Links:
- removed link camera_link
- added link head_camera_link
Joints:
- removed joint camera_joint
- added joint head_camera_joint: type fixed, parent torso_link, child head_camera_link, origin xyz=0.11109 0.01750 0.68789 rpy=-2.45672546 0 -1.5708
