Commit message: H1-2: MID-360 mount pitch 9.41 deg (0.1642 rad), measured on the real robot
livox_joint (torso_link -> livox_link) was rpy (0, 13.76 deg, 0). On the
real robot the lidar sits 9.41 deg nose-down (2026-10-17). Two independent
measurements over 21 bags agree to 0.1 deg:
- a gyro Wahba fit of /livox/imu against the torso IMU (blind to tilt and
  accelerometer bias);
- feet-flat FK gravity from the joint encoders. The same method reproduces
  the hand-tuned torso-IMU trim to 0.1-0.3 deg.

Roll and yaw stay 0 (both under 1 deg). The point frame reads 0.65 deg
lower than the IMU frame, which is below the policies' noise, so one
livox_link serves both.

Same value everywhere livox_link is defined:
- all 7 ros_assets URDFs;
- mujoco_assets/h1_2_magpie.xml, and robosuite_assets/robots/h1_2/robot.xml
  (regenerated by build_assets.py, only this line changes);
- isaac_assets h1_2_magpie USD: livox_joint localRot0 (physics layer) and
  livox_link xformOp:orient (base layer).

Co-Authored-By: Claude Opus 5.5 (1M context) <noreply@anthropic.com>

File: ros_assets/h1_2_handless.urdf (robot description, URDF)
Before this commit: robot h1_2, 36 links, 35 joints
Joints:
- joint livox_joint: origin xyz=0.04874 0 0.67980 rpy=0 0.24015730507441985 0 -> xyz=0.04874 0 0.67980 rpy=0 0.1642 0

File: ros_assets/h1_2_handless_ros.urdf (robot description, URDF)
Before this commit: robot h1_2, 36 links, 35 joints
Joints:
- joint livox_joint: origin xyz=0.04874 0 0.67980 rpy=0 0.24015730507441985 0 -> xyz=0.04874 0 0.67980 rpy=0 0.1642 0

File: ros_assets/h1_2_magpie.urdf (robot description, URDF)
Before this commit: robot h1_2_magpie, 54 links, 53 joints
Joints:
- joint livox_joint: origin xyz=0.04874 0 0.67980 rpy=0 0.24015730507441985 0 -> xyz=0.04874 0 0.67980 rpy=0 0.1642 0

File: ros_assets/h1_2_magpie_homie.urdf (robot description, URDF)
Before this commit: robot h1_2, 36 links, 35 joints
Joints:
- joint livox_joint: origin xyz=0.04874 0 0.67980 rpy=0 0.24015730507441985 0 -> xyz=0.04874 0 0.67980 rpy=0 0.1642 0

File: ros_assets/h1_2_magpie_ros.urdf (robot description, URDF)
Before this commit: robot h1_2_magpie, 54 links, 53 joints
Joints:
- joint livox_joint: origin xyz=0.04874 0 0.67980 rpy=0 0.24015730507441985 0 -> xyz=0.04874 0 0.67980 rpy=0 0.1642 0

Commit message: H1-2: MID-360 point frame and IMU chip as separate measured frames
The real MID-360's points and IMU disagree by 0.7 deg. Each frame now
carries its own measured pose, so consumers read the URDF instead of
keeping their own copies (FAST-LIO's extrinsic, the IMU lever arm, the
IMU trim):

- livox_link, the point frame: pitch 0.1531 rad (8.77 deg). From the floor
  plane in /livox/lidar against feet-flat FK.
- livox_imu_link (new), the frame of /livox/imu: child of livox_link.
  Position (0.011, -0.02329, 0.04412) m, Livox's IMU-in-lidar in the upright
  frame. rpy (-0.0016, 0.0119, 0) rad, the floor plane vs the accelerometer
  over 26 still windows (+-0.01 deg). The chip lands at 9.45 deg pitch in
  torso_link; a gyro fit against the torso IMU gives 9.51.

The MJCF's livox_imu_site moves to the same pose, so the sims' /livox/imu
carries the real lever arm and tilt. robosuite robot.xml is regenerated.
The USD gets livox_link's pose in both layers and a livox_imu_link Xform
under it; Isaac Lab's Imu accepts a prim with a rigid ancestor.

Co-Authored-By: Claude Opus 5.5 (1M context) <noreply@anthropic.com>

File: ros_assets/h1_2_handless.urdf (robot description, URDF)
Before this commit: robot h1_2, 36 links, 35 joints
Links:
- added link livox_imu_link
Joints:
- added joint livox_imu_joint: type fixed, parent livox_link, child livox_imu_link, origin xyz=0.011 -0.02329 0.04412 rpy=-0.0016 0.0119 0
- joint livox_joint: origin xyz=0.04874 0 0.67980 rpy=0 0.1642 0 -> xyz=0.04874 0 0.67980 rpy=0 0.1531 0

File: ros_assets/h1_2_handless_ros.urdf (robot description, URDF)
Before this commit: robot h1_2, 36 links, 35 joints
Links:
- added link livox_imu_link
Joints:
- added joint livox_imu_joint: type fixed, parent livox_link, child livox_imu_link, origin xyz=0.011 -0.02329 0.04412 rpy=-0.0016 0.0119 0
- joint livox_joint: origin xyz=0.04874 0 0.67980 rpy=0 0.1642 0 -> xyz=0.04874 0 0.67980 rpy=0 0.1531 0

File: ros_assets/h1_2_magpie.urdf (robot description, URDF)
Before this commit: robot h1_2_magpie, 54 links, 53 joints
Links:
- added link livox_imu_link
Joints:
- added joint livox_imu_joint: type fixed, parent livox_link, child livox_imu_link, origin xyz=0.011 -0.02329 0.04412 rpy=-0.0016 0.0119 0
- joint livox_joint: origin xyz=0.04874 0 0.67980 rpy=0 0.1642 0 -> xyz=0.04874 0 0.67980 rpy=0 0.1531 0

File: ros_assets/h1_2_magpie_homie.urdf (robot description, URDF)
Before this commit: robot h1_2, 36 links, 35 joints
Links:
- added link livox_imu_link
Joints:
- added joint livox_imu_joint: type fixed, parent livox_link, child livox_imu_link, origin xyz=0.011 -0.02329 0.04412 rpy=-0.0016 0.0119 0
- joint livox_joint: origin xyz=0.04874 0 0.67980 rpy=0 0.1642 0 -> xyz=0.04874 0 0.67980 rpy=0 0.1531 0

File: ros_assets/h1_2_magpie_ros.urdf (robot description, URDF)
Before this commit: robot h1_2_magpie, 54 links, 53 joints
Links:
- added link livox_imu_link
Joints:
- added joint livox_imu_joint: type fixed, parent livox_link, child livox_imu_link, origin xyz=0.011 -0.02329 0.04412 rpy=-0.0016 0.0119 0
- joint livox_joint: origin xyz=0.04874 0 0.67980 rpy=0 0.1642 0 -> xyz=0.04874 0 0.67980 rpy=0 0.1531 0
