Commit message: :bug: Fix *_graspgenx_frame to coincide with GraspGenX's magpie gripper base
A GraspGenX pose is executed by driving *_graspgenx_frame straight to it, so
that frame MUST be the gripper-BASE frame of GraspGenX's magpie model. It
wasn't: GraspGenX's magpie config.json puts the fingertip contact 0.1145763 m
along +Z from the base, but the frame sat at wrist x=0.085, making
graspgenx_frame -> grasp_frame only 0.113 - 0.032415 m short.

Every grasp therefore drove the jaws ~3.2 cm PAST the target: they closed on
each other and shoved the object instead of gripping it. x = 0.085 + 0.032415
= 0.117415 makes the base->fingertip span exactly 0.1145763, matching the
GraspGenX gripper model.

Co-Authored-By: Claude Opus 4.8 <noreply@anthropic.com>

File: ros_assets/h1_2_magpie_ros.urdf (robot description, URDF)
Before this commit: robot h1_2_magpie, 54 links, 53 joints
Joints:
- joint left_graspgenx_frame_joint: origin xyz=0.085 0 -0.001613 rpy=1.5708 0 1.5708 -> xyz=0.117415 0 -0.001613 rpy=1.5708 0 1.5708
- joint right_graspgenx_frame_joint: origin xyz=0.085 0 -0.001613 rpy=1.5708 0 1.5708 -> xyz=0.117415 0 -0.001613 rpy=1.5708 0 1.5708
