Commit message: g1: torso spheres that clear the hanging upper arms
The G1's hanging upper arms are 9 mm from the real torso at golem_upper_ik's
home (g1_description's meshes). The lab's three torso spheres followed the
torso's flanks, so the shoulder-yaw spheres sat 2.2 mm from them there and the
arm IK's self-collision keep-out had to drop to 2 mm.

The torso spheres are now a column on the midplane (torso z 0.061, 0.116,
0.212 m; r 0.078, 0.086, 0.102 m). Their sides stay 6-19 mm inside the flanks
from the waist to the chest, so at home every arm sphere clears the torso by
25 mm and the G1 keeps the H1-2's 20 mm keep-out. Elsewhere the column covers
the torso mesh about as well as the lab's spheres (at most 25 mm of mesh
outside it, against 22 mm). Sampled at the barrier's boundary, the arms come
within 2 mm of the real torso in 2 of 150 postures, against 22 of 150 with
the lab's spheres at 2 mm.

The SRDF is unchanged: no pair is disabled.

Co-Authored-By: Claude Opus 5.5 (1M context) <noreply@anthropic.com>
Claude-Session: https://claude.ai/code/session_01MezUeauFS9tKMgZKJxo1HC

File: g1/g1_sphere.urdf (robot description, URDF)
Before this commit: robot g1_29dof_rev_1_0, 63 links, 62 joints
Links:
- link torso_link_sphere1: geometry collision sphere radius=0.078; visual sphere radius=0.078
- link torso_link_sphere2: geometry collision sphere radius=0.086; visual sphere radius=0.086
- link torso_link_sphere3: geometry collision sphere radius=0.102; visual sphere radius=0.102
Joints:
- joint torso_link_to_torso_link_sphere1: origin xyz=0.005159590858966112 -0.001993038458749652 0.08828842639923096 rpy=0 0 0 -> xyz=0 0 0.061 rpy=0 0 0
- joint torso_link_to_torso_link_sphere2: origin xyz=0.0039655775763094425 -0.03270402550697327 0.21518424153327942 rpy=0 0 0 -> xyz=0 0 0.116 rpy=0 0 0
- joint torso_link_to_torso_link_sphere3: origin xyz=0.005717250518500805 0.029324715957045555 0.218731090426445 rpy=0 0 0 -> xyz=0.002 0 0.212 rpy=0 0 0
